Commit message: Working EKF Odometry

File: src/mensabot_description/urdf/mensabot.urdf.xacro (robot description, xacro)
@@ -223,5 +223,5 @@
   </gazebo>
   <joint name="camera_optical_joint" type="fixed">
-    <origin xyz="0 0 0" rpy="0 0 0"/>
+    <origin xyz="0 0 0" rpy="${-pi/2} 0 ${-pi/2}"/>
     <parent link="camera_link"/>
     <child link="camera_optical_frame"/>
